File: kicad/PCM3060-ESP32/PCM3060-ESP32.kicad_sch (KiCad schematic)
At the start: 4 parts

Commit message: gg
Parts:
- added C? (x2): .1uF, symbol Device:C
- added R? (x2): 330, symbol xenir:Resistor
Connections:
- net GND: now also U?.16 (SGND), C?.2, C?.2
- net RST: now reaches U?.15 (RST)
- net RST: now also U?.30 (IO17)
- net at U?.17 (VOUTR-): now also R?.1
- net at U?.18 (VOUTR+): now also R?.1
- new net: C?.1, R?.2 (x2)
Changed lines of the file:
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@@
+    (stroke (width 0) (type default) (color 0 0 0 0))
+  )
+  (wire (pts (xy 167.64 102.87) (xy 173.99 102.87))
+    (stroke (width 0) (type default) (color 0 0 0 0))
+  )
+  (wire (pts (xy 168.91 113.03) (xy 165.1 113.03))
+    (stroke (width 0) (type default) (color 0 0 0 0))
+  )
+  (wire (pts (xy 173.99 102.87) (xy 173.99 119.38))
+    (stroke (width 0) (type default) (color 0 0 0 0))
+  )
+  (wire (pts (xy 168.91 107.95) (xy 168.91 113.03))
     (stroke (width 0) (type default) (color 0 0 0 0))
   )
@@
     (stroke (width 0) (type default) (color 0 0 0 0))
   )
+  (wire (pts (xy 167.64 100.33) (xy 176.53 100.33))
+    (stroke (width 0) (type default) (color 0 0 0 0))
+  )
+  (wire (pts (xy 176.53 105.41) (xy 181.61 105.41))
+    (stroke (width 0) (type default) (color 0 0 0 0))
+  )
   (wire (pts (xy 120.65 77.47) (xy 133.35 77.47))
     (stroke (width 0) (type default) (color 0 0 0 0))
@@
     (stroke (width 0) (type default) (color 0 0 0 0))
   )
+  (wire (pts (xy 191.77 105.41) (xy 196.85 105.41))
+    (stroke (width 0) (type default) (color 0 0 0 0))
+  )
   (wire (pts (xy 107.95 96.52) (xy 114.3 96.52))
     (stroke (width 0) (type default) (color 0 0 0 0))
   )
+  (wire (pts (xy 173.99 119.38) (xy 181.61 119.38))
+    (stroke (width 0) (type default) (color 0 0 0 0))
+  )
   (wire (pts (xy 167.64 74.93) (xy 195.58 74.93))
     (stroke (width 0) (type default) (color 0 0 0 0))
   )
+  (wire (pts (xy 167.64 105.41) (xy 171.45 105.41))
+    (stroke (width 0) (type default) (color 0 0 0 0))
+  )
   (wire (pts (xy 107.95 71.12) (xy 123.19 71.12))
     (stroke (width 0) (type default) (color 0 0 0 0))
@@
     (stroke (width 0) (type default) (color 0 0 0 0))
   )
+  (wire (pts (xy 176.53 100.33) (xy 176.53 105.41))
+    (stroke (width 0) (type default) (color 0 0 0 0))
+  )
   (wire (pts (xy 120.65 73.66) (xy 120.65 77.47))
     (stroke (width 0) (type default) (color 0 0 0 0))
@@
     (stroke (width 0) (type default) (color 0 0 0 0))
   )
+  (wire (pts (xy 167.64 107.95) (xy 168.91 107.95))
+    (stroke (width 0) (type default) (color 0 0 0 0))
+  )
   (wire (pts (xy 127 90.17) (xy 127 68.58))
     (stroke (width 0) (type default) (color 0 0 0 0))
@@
   (wire (pts (xy 114.3 82.55) (xy 114.3 96.52))
     (stroke (width 0) (type default) (color 0 0 0 0))
+  )
+  (wire (pts (xy 191.77 119.38) (xy 196.85 119.38))
+    (stroke (width 0) (type default) (color 0 0 0 0))
+  )
+  (global_label "RST" (shape input) (at 165.1 113.03 180) (fields_autoplaced)
+    (effects (font (size 1.27 1.27)) (justify right))
+    (property "Intersheet References" "${INTERSHEET_REFS}" (id 0) (at 159.2398 113.1094 0)
+      (effects (font (size 1.27 1.27)) (justify right) hide)
+    )
+  )
+  (global_label "RST" (shape input) (at 107.95 93.98 0) (fields_autoplaced)
+    (effects (font (size 1.27 1.27)) (justify left))
+    (property "Intersheet References" "${INTERSHEET_REFS}" (id 0) (at 113.8102 93.9006 0)
+      (effects (font (size 1.27 1.27)) (justify left) hide)
+    )
   )
   (symbol (lib_id "xenir_v6:PCM3060") (at 149.86 68.58 0) (unit 1)
@@
     (pin "9")
   )
+  (symbol (lib_id "xenir:Resistor") (at 186.69 119.38 0) (unit 1)
+    (in_bom yes) (on_board yes) (fields_autoplaced)
+    (property "Reference" "R?" (id 0) (at 186.69 114.3 0)
+      (effects (font (size 0.7112 0.7112)))
+    )
+    (property "Value" "330" (id 1) (at 186.69 116.84 0)
+      (effects (font (size 0.7112 0.7112)))
+    )
+    (property "Footprint" "" (id 2) (at 186.69 121.92 0)
+      (effects (font (size 1.27 1.27)) hide)
+    )
+    (property "Datasheet" "" (id 3) (at 186.69 121.92 0)
+      (effects (font (size 1.27 1.27)) hide)
+    )
+    (pin "1")
+    (pin "2")
+  )
   (symbol (lib_id "power:GND") (at 195.58 77.47 0) (unit 1)
     (in_bom yes) (on_board yes) (fields_autoplaced)
@@
     )
     (pin "1")
+  )
+  (symbol (lib_id "Device:C") (at 196.85 123.19 0) (unit 1)
+    (in_bom yes) (on_board yes) (fields_autoplaced)
+    (property "Reference" "C?" (id 0) (at 200.66 121.9199 0)
+      (effects (font (size 1.27 1.27)) (justify left))
+    )
+    (property "Value" ".1uF" (id 1) (at 200.66 124.4599 0)
+      (effects (font (size 1.27 1.27)) (justify left))
+    )
+    (property "Footprint" "" (id 2) (at 197.8152 127 0)
+      (effects (font (size 1.27 1.27)) hide)
+    )
+    (property "Datasheet" "~" (id 3) (at 196.85 123.19 0)
+      (effects (font (size 1.27 1.27)) hide)
+    )
+    (pin "1")
+    (pin "2")
   )
   (symbol (lib_id "Device:C") (at 184.15 88.9 0) (unit 1)
@@
     (pin "1")
   )
+  (symbol (lib_id "xenir:Resistor") (at 186.69 105.41 0) (unit 1)
+    (in_bom yes) (on_board yes) (fields_autoplaced)
+    (property "Reference" "R?" (id 0) (at 186.69 100.33 0)
+      (effects (font (size 0.7112 0.7112)))
+    )
+    (property "Value" "330" (id 1) (at 186.69 102.87 0)
+      (effects (font (size 0.7112 0.7112)))
+    )
+    (property "Footprint" "" (id 2) (at 186.69 107.95 0)
+      (effects (font (size 1.27 1.27)) hide)
+    )
+    (property "Datasheet" "" (id 3) (at 186.69 107.95 0)
+      (effects (font (size 1.27 1.27)) hide)
+    )
+    (pin "1")
+    (pin "2")
+  )
+  (symbol (lib_id "power:GND") (at 196.85 113.03 0) (unit 1)
+    (in_bom yes) (on_board yes)
+    (property "Reference" "#PWR?" (id 0) (at 196.85 119.38 0)
+      (effects (font (size 1.27 1.27)) hide)
+    )
+    (property "Value" "GND" (id 1) (at 200.66 114.3 0))
+    (property "Footprint" "" (id 2) (at 196.85 113.03 0)
+      (effects (font (size 1.27 1.27)) hide)
+    )
+    (property "Datasheet" "" (id 3) (at 196.85 113.03 0)
+      (effects (font (size 1.27 1.27)) hide)
+    )
+    (pin "1")
+  )
   (symbol (lib_id "power:+5V") (at 175.26 85.09 0) (unit 1)
     (in_bom yes) (on_board yes) (fields_autoplaced)
@@
     )
     (property "Datasheet" "" (id 3) (at 175.26 85.09 0)
+      (effects (font (size 1.27 1.27)) hide)
+    )
+    (pin "1")
+  )
+  (symbol (lib_id "power:GND") (at 171.45 105.41 0) (unit 1)
+    (in_bom yes) (on_board yes) (fields_autoplaced)
+    (property "Reference" "#PWR?" (id 0) (at 171.45 111.76 0)
+      (effects (font (size 1.27 1.27)) hide)
+    )
+    (property "Value" "GND" (id 1) (at 171.45 110.49 0))
+    (property "Footprint" "" (id 2) (at 171.45 105.41 0)
+      (effects (font (size 1.27 1.27)) hide)
+    )
+    (property "Datasheet" "" (id 3) (at 171.45 105.41 0)
+      (effects (font (size 1.27 1.27)) hide)
+    )
+    (pin "1")
+  )
+  (symbol (lib_id "power:GND") (at 196.85 127 0) (unit 1)
+    (in_bom yes) (on_board yes)
+    (property "Reference" "#PWR?" (id 0) (at 196.85 133.35 0)
+      (effects (font (size 1.27 1.27)) hide)
+    )
+    (property "Value" "GND" (id 1) (at 200.66 128.27 0))
+    (property "Footprint" "" (id 2) (at 196.85 127 0)
+      (effects (font (size 1.27 1.27)) hide)
+    )
+    (property "Datasheet" "" (id 3) (at 196.85 127 0)
       (effects (font (size 1.27 1.27)) hide)
     )
@@
     (pin "1")
   )
+  (symbol (lib_id "Device:C") (at 196.85 109.22 0) (unit 1)
+    (in_bom yes) (on_board yes) (fields_autoplaced)
+    (property "Reference" "C?" (id 0) (at 200.66 107.9499 0)
+      (effects (font (size 1.27 1.27)) (justify left))
+    )
+    (property "Value" ".1uF" (id 1) (at 200.66 110.4899 0)
+      (effects (font (size 1.27 1.27)) (justify left))
+    )
+    (property "Footprint" "" (id 2) (at 197.8152 113.03 0)
+      (effects (font (size 1.27 1.27)) hide)
+    )
+    (property "Datasheet" "~" (id 3) (at 196.85 109.22 0)
+      (effects (font (size 1.27 1.27)) hide)
+    )
+    (pin "1")
+    (pin "2")
+  )
   (sheet_instances
     (path "/" (page "1"))
@@
       (reference "#PWR?") (unit 1) (value "GND") (footprint "")
     )
+    (path "/a1c34d60-ffa3-4b59-b8ca-cfb3e8601fab"
+      (reference "#PWR?") (unit 1) (value "GND") (footprint "")
+    )
     (path "/a72b7a1d-3e61-430a-890a-c5c687423317"
       (reference "#PWR?") (unit 1) (value "+5V") (footprint "")
     )
+    (path "/aa5971bf-473e-4143-b89d-10ceba7f1414"
+      (reference "#PWR?") (unit 1) (value "GND") (footprint "")
+    )
+    (path "/bb6a9044-97ef-4952-b648-6ccf47b4e959"
+      (reference "#PWR?") (unit 1) (value "GND") (footprint "")
+    )
     (path "/e719144f-f31e-41d8-b88a-ac5669e89d2c"
       (reference "#PWR?") (unit 1) (value "GND") (footprint "")
     )
+    (path "/2ab9f9ab-f431-49b1-99af-5c7f9e02bacd"
+      (reference "C?") (unit 1) (value ".1uF") (footprint "")
+    )
     (path "/46dbed5d-37bb-4ad7-b00f-9b748fbab36b"
       (reference "C?") (unit 1) (value ".1uF") (footprint "")
@@
       (reference "C?") (unit 1) (value ".1uF") (footprint "")
     )
+    (path "/f81284d2-d377-4f45-b26b-f1127fb653d0"
+      (reference "C?") (unit 1) (value ".1uF") (footprint "")
+    )
+    (path "/17dfde56-c6fe-4216-b23c-247ae202a84b"
+      (reference "R?") (unit 1) (value "330") (footprint "")
+    )
+    (path "/98df8625-3ce3-4cd7-abd1-655dc53585e4"
+      (reference "R?") (unit 1) (value "330") (footprint "")
+    )
     (path "/0b7e1aca-1046-4752-acb4-58ac47ece09b"

Commit message: gg
Parts:
- added C3, C4: 4.7uF, symbol Device:C_Polarized
- gave numbers to parts that had none: 8
Connections:
- net at U2.25 (VINL): now also C4.1
- net at U2.26 (VINR): now also C3.1
- new net INPUT_L: C4.2
- new net INPUT_R: C3.2
